Commit message: Added the RTAB-Map launch file for localization

File: src/my_robot/urdf/my_robot.xacro (robot description, xacro)
@@ -127,4 +127,6 @@
         </visual>
     </link>
+    <link name="camera_link_optical">
+    </link>
     <link name='hokuyo'>
         <inertial>
@@ -187,6 +189,4 @@
         <child link="camera_link_optical"/>
     </joint>
-    <link name="camera_link_optical">
-    </link>
     <gazebo reference="left_wheel">
         <material>Gazebo/DarkGray</material>

Commit message: Fixed the kinect camera issue affecting SLAM

File: src/my_robot/urdf/my_robot.xacro (robot description, xacro)
@@ -175,5 +175,4 @@
     </joint>
     <joint type="fixed" name="hokuyo_joint">
-        <!-- <origin xyz="0.15 0 0.1" rpy="0 0 0"/> -->
         <origin xyz="0 0 0.1" rpy="0 0 0"/>
         <child link="hokuyo"/>
@@ -184,6 +183,5 @@
     </joint>
     <joint name="camera_optical_joint" type="fixed">
-        <!-- <origin xyz="0 0 0" rpy="-1.5707 0 -1.5707"/>  -->
-        <origin xyz="0 0 0" rpy="0 0 0"/>
+        <origin xyz="0 0 0" rpy="-1.5707 0 -1.5707"/>
         <parent link="camera"/>
         <child link="camera_link_optical"/>
